File: docs/elec/alim5v/alim5V.sch (KiCad schematic (older format))
At the start: 7 parts, among them P1 GND Ardui, P2 5V out, P3 MD49, P4 Charg, P5 Batt, SW1 SW, U1 UEI30-050-Q12P-C

Commit message: ajout connecteur carte puissance
Parts:
- added P6: 5V out AUX, Pin_Headers:Pin_Header_Angled_1x02, symbol CONN_01X02
- added P7: AUX, robair:Bornier5mm, symbol CONN_01X02
Connections:
- net GND24: now also P7.1 (P1)
- net GND5: now also P6.2 (P2)
- net at P3.2 (P2), SW1.1, U1.1 (Vin+): now also P7.2 (P2)
- net at P2.1 (P1), U1.4 (Vout+): now also P6.1 (P1)
Changed lines of the file:
@@
 $EndComp
 Wire Wire Line
-	5800 3600 6200 3600
+	6200 3600 5800 3600
 Wire Wire Line
-	5800 3700 6100 3700
+	6100 3700 5800 3700
 Wire Wire Line
 	4400 3600 4200 3600
@@
 	4200 3100 4300 3100
 Wire Wire Line
-	4300 3100 4300 3600
+	4300 3100 4300 3900
 Connection ~ 4300 3600
 Text Label 5850 3600 0    60   ~ 0
@@
 	7900 3450 7550 3450
 Wire Wire Line
-	6200 3600 6200 3350
+	6200 2900 6200 3600
 Connection ~ 7800 3350
 Wire Wire Line
@@
 	7350 3100 6050 3100
 Wire Wire Line
-	6100 3700 6100 3100
+	6100 2800 6100 3700
 Connection ~ 6100 3100
+$Comp
+L CONN_01X02 P7
+U 1 1 585255F2
+P 5850 2850
+F 0 "P7" H 5850 3000 50  0000 C CNN
+F 1 "AUX" V 5950 2850 50  0000 C CNN
+F 2 "robair:Bornier5mm" H 5850 2850 50  0001 C CNN
+F 3 "" H 5850 2850 50  0000 C CNN
+	1    5850 2850
+	-1   0    0    1
+$EndComp
+$Comp
+L CONN_01X02 P6
+U 1 1 58525622
+P 4000 3950
+F 0 "P6" H 4000 4100 50  0000 C CNN
+F 1 "5V out AUX" V 4100 3950 50  0000 C CNN
+F 2 "Pin_Headers:Pin_Header_Angled_1x02" H 4000 3950 50  0001 C CNN
+F 3 "" H 4000 3950 50  0000 C CNN
+	1    4000 3950
+	-1   0    0    1
+$EndComp
+Wire Wire Line
+	6050 2900 6200 2900
+Wire Wire Line
+	6050 2800 6100 2800
+Wire Wire Line
+	4300 3900 4200 3900
+Wire Wire Line
+	4200 4000 4350 4000
+Wire Wire Line
+	4350 4000 4350 3700
+Connection ~ 4350 3700
 $EndSCHEMATC
